File: sound_card/sound_card.kicad_pcb (KiCad board)
At the start: 2 copper layers, 100 x 78 mm, 29 parts, among them IC1 SN74HCT138N, J1 Conn1, J2 Right Channel, J3 ~{WAIT} State Select, J4 Left Channel, J5 AudioJack3, U1 AY-3-8910, U2 74HCT00, U3 74LS163, U4 74HCT04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

Commit message: Added address map to schematic and pcb silkscreen
Other:
- board text added: "3.5mm"
- board text added: "Address Map: Read/Write - 0x00 Latch (WR) - 0x01"
Changed lines of the file:
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@@
 		(tags "TRS audio jack stereo horizontal")
 		(property "Reference" "J5"
-			(at 0 -8.8 90)
+			(at 5.26 -9.175 90)
 			(layer "F.SilkS")
 			(effects
@@
 		)
 	)
+	(gr_text "3.5mm"
+		(at 186.25 76.111191 270)
+		(layer "F.SilkS")
+		(effects
+			(font
+				(size 1 1)
+				(thickness 0.15)
+			)
+			(justify left bottom)
+		)
+	)
 	(gr_text "74HCT00"
 		(at 149.125 113.45 90)
@@
 		(layer "F.SilkS")
 		(effects
+			(font
+				(size 1 1)
+				(thickness 0.15)
+			)
+			(justify left bottom)
+		)
+	)
+	(gr_text "Address Map:\nRead/Write - 0x00\nLatch (WR) - 0x01"
+		(at 168.275 77.525 0)
+		(layer "F.SilkS")
+		(effects
