File: sound_card/sound_card.kicad_sch (KiCad schematic)
At the start: 29 parts, among them IC1 SN74HCT138N, J1 Conn1, J2 Right Channel, J3 ~{WAIT} State Select, J4 Left Channel, J5 AudioJack3, U1 AY-3-8910, U2 74HCT00, U3 74LS163, U4 74HCT04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

Commit message: Added address map to schematic and pcb silkscreen
Other:
- note added: "Read/Write - 0x00 Latch (WR) - 0x01"
Changed lines of the file:
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@@
 	(rectangle
 		(start 218.44 124.46)
-		(end 313.69 170.18)
+		(end 312.42 176.53)
 		(stroke
 			(width 0)
@@
 			)
 		)
+	)
+	(text "Read/Write - 0x00\nLatch (WR) - 0x01"
+		(exclude_from_sim no)
+		(at 265.938 170.942 0)
+		(effects
+			(font
+				(size 2 2)
+			)
+		)

Commit message: Fixed mislabeled title on schematic
Other:
- title: Kludge CPU Card -> Kludge Sound Card
Changed lines of the file:
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@@
 	(paper "B")
 	(title_block
-		(title "Kludge CPU Card")
+		(title "Kludge Sound Card")
 		(rev "1.0")
 	)
