File: video_card/video_card.kicad_pcb (KiCad board)
At the start: 2 copper layers, 100 x 85 mm, 22 parts, among them J1 Bus, J2 DE15_Receptacle_HighDensity, J3 H_SYNC_TEST, J4 V_SYNC_TEST, J5 VSYNC_INT_EN, J6 INT_EN, U1 Upduino v3.1, U2 25.175 MHz, U3 SN74LVC4245A, U4 SN74LVC4245A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

Commit message: Swapped out '4245' on the INT signal to a more simple transistor circuit
Parts:
- removed J5: VSYNC_INT_EN, Connector_PinHeader_2.54mm:PinHeader_2x01_P2.54mm_Vertical
- removed J6: INT_EN, Connector_PinHeader_2.54mm:PinHeader_2x01_P2.54mm_Vertical
- removed R10: 1K, Resistor_THT:R_Axial_DIN0207_L6.3mm_D2.5mm_P10.16mm_Horizontal
- removed U6: SN74LVC4245A, Z80 Parts:SN74LVC4245A
- added Q1: 2N2222, Package_TO_SOT_THT:TO-92, F.Cu at (121.1, 79.7)
- J3: footprint Connector_PinHeader_2.54mm:PinHeader_1x01_P2.54mm_Vertical -> Connector_PinHeader_2.54mm:PinHeader_1x02_P2.54mm_Vertical
- J4: value V_SYNC_TEST -> INT_EN; footprint Connector_PinHeader_2.54mm:PinHeader_1x01_P2.54mm_Vertical -> Connector_PinHeader_2.54mm:PinHeader_1x03_P2.54mm_Vertical
- U3, U4: footprint Z80 Parts:SN74LVC4245A -> Z80 Parts:SN74LVC4245ADWR
- moved J4 47.7 mm to (132.5, 85.0), turned to 90 degrees
- moved R9 40.1 mm to (117.3, 85.2), turned to 0 degrees
- moved J2 5.08 mm to (187.4, 72.8)
- moved J3 5.08 mm to (180.2, 77.5)
- moved R1 5.08 mm to (172.8, 86.4)
- moved R2 5.08 mm to (169.7, 86.4)
- moved R3 5.08 mm to (166.6, 86.4)
- moved R4 5.08 mm to (163.4, 86.4)
- moved R5 5.08 mm to (160.3, 86.4)
- moved R6 5.08 mm to (157.2, 86.4)
- moved R7 5.08 mm to (154.1, 86.4)
- moved R8 5.08 mm to (150.9, 86.4)
- moved U1 5.08 mm to (127.4, 105.7)
- moved U2 5.08 mm to (188.8, 100.0)
- moved U4 5.01 mm to (168.8, 124.4)
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Connections:
- J1 pad 23: INT -> ~{INT}
- J1 pad 25: unconnected-(J1-Pin_25-Pad25) -> ~{NMI}
- J4 pad 1: /V_SYNC -> ~{INT}
- R9 pad 2: INT -> V_INT
- U1 pad 18: /V_D6 -> unconnected-(U1-GPIO_37_G1-Pad18)
- U1 pad 19: /V_D7 -> /V_D6
- U1 pad 20: /V_ADDR3 -> /V_D7
- U1 pad 21: /V_ADDR2 -> /V_ADDR3
- U1 pad 22: /V_ADDR1 -> /V_ADDR2
- U1 pad 23: /V_ADDR0 -> /V_ADDR1
- U1 pad 24: unconnected-(U1-GPIO_28-Pad24) -> /V_ADDR0
- U1 pad 39: /~{BUS_INT} -> V_INT
Routing:
- net ~{INT}: track 0.00 -> 68.6 mm, vias 0 -> 2
- net ~{NMI}: track 0.00 -> 64.3 mm, vias 0 -> 1
- net INT: track 44.4 -> 0.00 mm, vias 2 -> 0
- net V_INT: track 59.2 -> 17.8 mm, vias 2 -> 0
- net GND: track 358.5 -> 322.2 mm, vias 17 -> 10
- net /V_SYNC: track 103.3 -> 70.6 mm
- net VCC: track 179.0 -> 199.5 mm, vias 3 -> 8
- net Net-(J4-Pin_2): track 0.00 -> 16.2 mm
- net /V_ADDR0: track 6.40 -> 19.5 mm, vias 0 -> 2
- net /V_ADDR1: track 5.62 -> 18.3 mm, vias 0 -> 2
- net /~{BUS_INT}: track 11.9 -> 0.00 mm
- net /V_D6: track 11.2 -> 22.1 mm, vias 0 -> 2
- net 3.3V: track 68.4 -> 57.7 mm, vias 3 -> 4
- net /V_ADDR2: track 6.40 -> 17.0 mm, vias 0 -> 2
- net /A3: track 40.3 -> 30.0 mm
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Other:
- board size 100 x 85 mm -> 100 x 90.1 mm
- board text added: "2N2222"
- board text added: "INT"
- board text added: "Kludge Video Card v1.1"
- board text added: "NMI"
- board text removed: "VSYNC_INT"
